File: pcb/remote-controller-board/remote-controller-board.kicad_sch (KiCad schematic)
At the start: 6 parts, among them J1 Conn_01x07, J2 Conn_01x05, SW1 SW_Push, SW2 SW_Push, SW3 SW_Push, SW4 SW_Push

Commit message: New PCB & case
Parts:
- removed SW1, SW2, SW3, SW4: SW_Push, Button_Switch_SMD:Panasonic_EVQPUM_EVQPUD, symbol Switch:SW_Push
- J2: footprint Connector_PinSocket_2.54mm:PinSocket_1x05_P2.54mm_Vertical -> Custom:Conn_01x05
Changed lines of the file:
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@@
-    )
-  )
-  (global_label "RE3" (shape input) (at 114.3 59.69 180) (fields_autoplaced)
-    (effects (font (size 1.27 1.27)) (justify right))
-    (property "Intersheetrefs" "${INTERSHEET_REFS}" (at 107.7657 59.69 0)
-      (effects (font (size 1.27 1.27)) (justify right) hide)
-    )
-  )
-  (global_label "GND2" (shape input) (at 124.46 59.69 0) (fields_autoplaced)
-    (effects (font (size 1.27 1.27)) (justify left))
-    (property "Intersheetrefs" "${INTERSHEET_REFS}" (at 132.4458 59.69 0)
-      (effects (font (size 1.27 1.27)) (justify left) hide)
-    )
-  )
-  (global_label "GND2" (shape input) (at 124.46 71.12 0) (fields_autoplaced)
-    (effects (font (size 1.27 1.27)) (justify left))
-    (property "Intersheetrefs" "${INTERSHEET_REFS}" (at 132.4458 71.12 0)
-      (effects (font (size 1.27 1.27)) (justify left) hide)
     )
   )
@@
     (effects (font (size 1.27 1.27)) (justify right))
     (property "Intersheetrefs" "${INTERSHEET_REFS}" (at 173.8057 44.45 0)
-      (effects (font (size 1.27 1.27)) (justify right) hide)
-    )
-  )
-  (global_label "GND2" (shape input) (at 124.46 36.83 0) (fields_autoplaced)
-    (effects (font (size 1.27 1.27)) (justify left))
-    (property "Intersheetrefs" "${INTERSHEET_REFS}" (at 132.4458 36.83 0)
-      (effects (font (size 1.27 1.27)) (justify left) hide)
-    )
-  )
-  (global_label "RE4" (shape input) (at 114.3 71.12 180) (fields_autoplaced)
-    (effects (font (size 1.27 1.27)) (justify right))
-    (property "Intersheetrefs" "${INTERSHEET_REFS}" (at 107.7657 71.12 0)
       (effects (font (size 1.27 1.27)) (justify right) hide)
     )
@@
     )
   )
-  (global_label "RE1" (shape input) (at 114.3 36.83 180) (fields_autoplaced)
-    (effects (font (size 1.27 1.27)) (justify right))
-    (property "Intersheetrefs" "${INTERSHEET_REFS}" (at 107.7657 36.83 0)
-      (effects (font (size 1.27 1.27)) (justify right) hide)
-    )
-  )
   (global_label "RE1" (shape input) (at 180.34 36.83 180) (fields_autoplaced)
     (effects (font (size 1.27 1.27)) (justify right))
     (property "Intersheetrefs" "${INTERSHEET_REFS}" (at 173.8057 36.83 0)
-      (effects (font (size 1.27 1.27)) (justify right) hide)
-    )
-  )
-  (global_label "GND2" (shape input) (at 124.46 48.26 0) (fields_autoplaced)
-    (effects (font (size 1.27 1.27)) (justify left))
-    (property "Intersheetrefs" "${INTERSHEET_REFS}" (at 132.4458 48.26 0)
-      (effects (font (size 1.27 1.27)) (justify left) hide)
-    )
-  )
-  (global_label "RE2" (shape input) (at 114.3 48.26 180) (fields_autoplaced)
-    (effects (font (size 1.27 1.27)) (justify right))
-    (property "Intersheetrefs" "${INTERSHEET_REFS}" (at 107.7657 48.26 0)
       (effects (font (size 1.27 1.27)) (justify right) hide)
     )
@@
     )
   )
-  (symbol (lib_id "Switch:SW_Push") (at 119.38 36.83 0) (unit 1)
-    (in_bom yes) (on_board yes) (dnp no) (fields_autoplaced)
-    (property "Reference" "SW1" (at 119.38 29.21 0)
-      (effects (font (size 1.27 1.27)))
-    )
-    (property "Value" "SW_Push" (at 119.38 31.75 0)
-      (effects (font (size 1.27 1.27)))
-    )
-    (property "Footprint" "Button_Switch_SMD:Panasonic_EVQPUM_EVQPUD" (at 119.38 31.75 0)
-      (effects (font (size 1.27 1.27)) hide)
-    )
-    (property "Datasheet" "~" (at 119.38 31.75 0)
-      (effects (font (size 1.27 1.27)) hide)
-    )
-    (pin "1")
-    (pin "2")
-    (instances
-      (project "remote-controller-board"
-        (path "/b41e7c80-a689-474c-b8df-401c60d9e215"
-          (reference "SW1") (unit 1)
-        )
-      )
-      (project "pcb"
-        (path "/be9b543b-b294-4f79-a0ab-4924c207a091"
-          (reference "SW1") (unit 1)
-        )
-      )
-      (project "main-board"
-        (path "/e93d6aa3-928d-4df9-b25b-21169669388b"
-          (reference "SW1") (unit 1)
-        )
-      )
-    )
-  )
   (symbol (lib_id "Connector_Generic:Conn_01x05") (at 185.42 41.91 0) (unit 1)
     (in_bom yes) (on_board yes) (dnp no) (fields_autoplaced)
@@
       (effects (font (size 1.27 1.27)) (justify left))
     )
-    (property "Footprint" "Connector_PinSocket_2.54mm:PinSocket_1x05_P2.54mm_Vertical" (at 185.42 41.91 0)
+    (property "Footprint" "Custom:Conn_01x05" (at 185.42 41.91 0)
       (effects (font (size 1.27 1.27)) hide)
     )
@@
         )
       )
-    )
-  )
-  (symbol (lib_id "Switch:SW_Push") (at 119.38 71.12 0) (unit 1)
-    (in_bom yes) (on_board yes) (dnp no) (fields_autoplaced)
-    (property "Reference" "SW4" (at 119.38 63.5 0)
-      (effects (font (size 1.27 1.27)))
-    )
-    (property "Value" "SW_Push" (at 119.38 66.04 0)
-      (effects (font (size 1.27 1.27)))
-    )
-    (property "Footprint" "Button_Switch_SMD:Panasonic_EVQPUM_EVQPUD" (at 119.38 66.04 0)
-      (effects (font (size 1.27 1.27)) hide)
-    )
-    (property "Datasheet" "~" (at 119.38 66.04 0)
-      (effects (font (size 1.27 1.27)) hide)
-    )
-    (pin "1")
-    (pin "2")
-    (instances
-      (project "remote-controller-board"
-        (path "/b41e7c80-a689-474c-b8df-401c60d9e215"
-          (reference "SW4") (unit 1)
-        )
-      )
-      (project "pcb"
-        (path "/be9b543b-b294-4f79-a0ab-4924c207a091"
-          (reference "SW1") (unit 1)
-        )
-      )
-      (project "main-board"
-        (path "/e93d6aa3-928d-4df9-b25b-21169669388b"
-          (reference "SW1") (unit 1)
-        )
-      )
-    )
-  )
-  (symbol (lib_id "Switch:SW_Push") (at 119.38 59.69 0) (unit 1)
-    (in_bom yes) (on_board yes) (dnp no) (fields_autoplaced)
-    (property "Reference" "SW3" (at 119.38 52.07 0)
-      (effects (font (size 1.27 1.27)))
-    )
-    (property "Value" "SW_Push" (at 119.38 54.61 0)
-      (effects (font (size 1.27 1.27)))
-    )
-    (property "Footprint" "Button_Switch_SMD:Panasonic_EVQPUM_EVQPUD" (at 119.38 54.61 0)
-      (effects (font (size 1.27 1.27)) hide)
-    )
-    (property "Datasheet" "~" (at 119.38 54.61 0)
-      (effects (font (size 1.27 1.27)) hide)
-    )
-    (pin "1")
-    (pin "2")
-    (instances
-      (project "remote-controller-board"
-        (path "/b41e7c80-a689-474c-b8df-401c60d9e215"
-          (reference "SW3") (unit 1)
-        )
-      )
-      (project "pcb"
-        (path "/be9b543b-b294-4f79-a0ab-4924c207a091"
-          (reference "SW1") (unit 1)
-        )
-      )
-      (project "main-board"
-        (path "/e93d6aa3-928d-4df9-b25b-21169669388b"
-          (reference "SW1") (unit 1)
-        )
-      )
-    )
-  )
-  (symbol (lib_id "Switch:SW_Push") (at 119.38 48.26 0) (unit 1)
-    (in_bom yes) (on_board yes) (dnp no) (fields_autoplaced)
-    (property "Reference" "SW2" (at 119.38 40.64 0)
-      (effects (font (size 1.27 1.27)))
-    )
-    (property "Value" "SW_Push" (at 119.38 43.18 0)
-      (effects (font (size 1.27 1.27)))
-    )
-    (property "Footprint" "Button_Switch_SMD:Panasonic_EVQPUM_EVQPUD" (at 119.38 43.18 0)
-      (effects (font (size 1.27 1.27)) hide)
-    )
-    (property "Datasheet" "~" (at 119.38 43.18 0)
-      (effects (font (size 1.27 1.27)) hide)
-    )
-    (pin "1")
-    (pin "2")
-    (instances
-      (project "remote-controller-board"
-        (path "/b41e7c80-a689-474c-b8df-401c60d9e215"
-          (reference "SW2") (unit 1)
-        )
-      )
-      (project "pcb"
-        (path "/be9b543b-b294-4f79-a0ab-4924c207a091"
-          (reference "SW1") (unit 1)
-        )
-      )
-      (project "main-board"
-        (path "/e93d6aa3-928d-4df9-b25b-21169669388b"
-          (reference "SW1") (unit 1)
-        )
-      )
